File: KiCad/window-sensor.kicad_pcb (KiCad board)
At the start: 2 copper layers, 82.5 x 22.4 mm, 19 parts, among them J1 Conn_01x05_Male, U3 74HC86

Commit message: Circuit corrected. Pullup now at GPIO0 instead of GPIO2.
Connections:
- ESP-12E1 pad 17: Net-(10k-3-Pad1) -> Net-(ESP-12E1-Pad17)
- ESP-12E1 pad 18: Net-(ESP-12E1-Pad18) -> Net-(10k-3-Pad1)
- FLASH1 pad 1: Net-(ESP-12E1-Pad18) -> Net-(10k-3-Pad1)
- J1 pad 3: Net-(ESP-12E1-Pad18) -> Net-(10k-3-Pad1)
- U3 pad 14: +3V3 -> (no net)
- U3 pad 7: GND -> (no net)
- U3 pad 9: GND -> (no net)
Routing:
- net Net-(ESP-12E1-Pad18): track 79.6 -> 0.00 mm, vias 1 -> 0
- net Net-(10k-3-Pad1): track 22.9 -> 100.2 mm, vias 2 -> 3
Other:
- board text added: "Window-Sensor v1.2"
- board text removed: "Window-Sensor v1.1"
